Commit message: almost working sim with a few weird issues with some weird physics. URDF had to be ultered for the sim so will need to be verified again with the robot
Made-with: Cursor

File: src/create_robot/create_description/urdf/rectangular_robot.urdf.xacro (robot description, xacro)
@@ -34,5 +34,5 @@
   <!-- Note: Rear wheels are forward by one wheel radius (origin is between rear wheels) -->
   <!-- Caster wheel properties -->
-  <xacro:property name="caster_radius" value="0.075" />
+  <xacro:property name="caster_radius" value="0.12" />
   <xacro:property name="caster_mass" value="0.5" />
   <!-- Caster at front of robot (base extends from x=0 to x=base_length, center at base_length/2) -->
@@ -72,4 +72,6 @@
       <origin xyz="${x} ${y} ${z}" rpy="0 0 0"/>
       <axis xyz="${axis_xyz}"/>
+      <!-- Stronger damping to suppress residual idle creep in Gazebo Classic. -->
+      <dynamics damping="0.5" friction="0.0"/>
     </joint>
   </xacro:macro>
@@ -78,6 +80,6 @@
   <link name="base_link">
     <visual>
-      <!-- Base extends from z=0 (ground) to z=base_height, centered at base_length/2 forward -->
-      <origin xyz="${base_length/2} 0 ${base_height/2}" rpy="0 0 0"/>
+      <!-- In simulation, keep chassis above ground by wheel radius to avoid floor dragging. -->
+      <origin xyz="${base_length/2} 0 ${wheel_radius + base_height/2}" rpy="0 0 0"/>
       <geometry>
         <box size="${base_length} ${base_width} ${base_height}"/>
@@ -86,5 +88,5 @@
     </visual>
     <collision>
-      <origin xyz="${base_length/2} 0 ${base_height/2}" rpy="0 0 0"/>
+      <origin xyz="${base_length/2} 0 ${wheel_radius + base_height/2}" rpy="0 0 0"/>
       <geometry>
         <box size="${base_length} ${base_width} ${base_height}"/>
@@ -92,12 +94,19 @@
     </collision>
     <inertial>
-      <origin xyz="${base_length/2} 0 ${base_height/2}" rpy="0 0 0"/>
+      <origin xyz="${base_length/2} 0 ${wheel_radius + base_height/2}" rpy="0 0 0"/>
       <mass value="${base_mass}"/>
       <inertia ixx="1.0" ixy="0" ixz="0" iyy="1.0" iyz="0" izz="1.0"/>
     </inertial>
   </link>
-  <!-- Rear wheels: classic diff-drive (+Y left, -Y right). Required for correct turn animation in RViz; both +Y makes straight OK but reverses both wheels when turning. -->
-  <xacro:wheel name="left_rear_wheel" x="${wheel_radius}" y="${wheel_separation/2}" z="0" axis_xyz="0 1 0"/>
-  <xacro:wheel name="right_rear_wheel" x="${wheel_radius}" y="${-wheel_separation/2}" z="0" axis_xyz="0 -1 0"/>
+  <!-- Add small body damping so the chassis settles at idle in simulation. -->
+  <gazebo reference="base_link">
+    <velocity_decay>
+      <linear>1.0</linear>
+      <angular>1.0</angular>
+    </velocity_decay>
+  </gazebo>
+  <!-- Rear wheels for Gazebo diff-drive: keep both joint axes aligned (+Y) so forward cmd drives straight. -->
+  <xacro:wheel name="left_rear_wheel" x="${wheel_radius}" y="${wheel_separation/2}" z="${wheel_radius}" axis_xyz="0 1 0"/>
+  <xacro:wheel name="right_rear_wheel" x="${wheel_radius}" y="${-wheel_separation/2}" z="${wheel_radius}" axis_xyz="0 1 0"/>
   <!-- Front Caster Wheel -->
   <link name="front_caster_wheel">
@@ -125,6 +134,36 @@
     <child link="front_caster_wheel"/>
     <!-- Caster at front of robot, at ground level -->
-    <origin xyz="${caster_x_offset} 0 0" rpy="0 0 0"/>
+    <origin xyz="${caster_x_offset} 0 ${caster_radius}" rpy="0 0 0"/>
   </joint>
+  <!-- Front caster with moderate contact (avoid injecting forward creep). -->
+  <gazebo reference="front_caster_wheel">
+    <mu1>0.05</mu1>
+    <mu2>0.05</mu2>
+    <kp>1000000.0</kp>
+    <kd>1.0</kd>
+    <minDepth>0.001</minDepth>
+    <maxVel>0.0</maxVel>
+  </gazebo>
+  <!-- Rear drive wheel contact tuning: high traction, low slip. -->
+  <gazebo reference="left_rear_wheel">
+    <mu1>1.5</mu1>
+    <mu2>1.5</mu2>
+    <slip1>0.0</slip1>
+    <slip2>0.0</slip2>
+    <kp>1000000.0</kp>
+    <kd>1.0</kd>
+    <minDepth>0.001</minDepth>
+    <maxVel>0.0</maxVel>
+  </gazebo>
+  <gazebo reference="right_rear_wheel">
+    <mu1>1.5</mu1>
+    <mu2>1.5</mu2>
+    <slip1>0.0</slip1>
+    <slip2>0.0</slip2>
+    <kp>1000000.0</kp>
+    <kd>1.0</kd>
+    <minDepth>0.001</minDepth>
+    <maxVel>0.0</maxVel>
+  </gazebo>
   <!-- Sweeping Wheel (parallel to floor - horizontal cylinder) -->
   <link name="sweeping_wheel">
@@ -151,6 +190,6 @@
     <parent link="base_link"/>
     <child link="sweeping_wheel"/>
-    <!-- Sweep wheel at front of robot, at ground level -->
-    <origin xyz="${sweep_wheel_x} ${sweep_wheel_y} 0" rpy="0 0 0"/>
+    <!-- Keep sweeper clear of floor contact in simulation. -->
+    <origin xyz="${sweep_wheel_x} ${sweep_wheel_y} ${sweep_wheel_radius}" rpy="0 0 0"/>
   </joint>
   <!-- Base Footprint (for navigation) - positioned at origin between rear wheels -->
@@ -163,9 +202,38 @@
     <origin xyz="${wheel_radius} 0 0" rpy="0 0 0"/>
   </joint>
-  <!-- Lidar positioned above rear wheels on top of body -->
-  <!-- Position: x=wheel_radius (where rear wheels are), y=0 (center), z=base_height (top of base) + half lidar height (0.02m) -->
-  <!-- Note: base_link origin is at (0, 0, 0), rear wheels are at x=wheel_radius (0.12m), base extends from z=0 to z=base_height (0.1m) -->
-  <!-- Lidar center sits at top of base + half lidar height (0.02m) = 0.12m -->
-  <xacro:lidar parent_link="base_link" x="${wheel_radius}" y="0" z="${base_height + 0.02}"/>
+  <!-- Keep lidar directly over rear axle (real robot mounting), raise height to reduce wheel returns. -->
+  <xacro:lidar parent_link="base_link" x="${wheel_radius}" y="0" z="${base_height + 0.25}"/>
+  <!-- Gazebo diff-drive for Classic simulation -->
+  <gazebo>
+    <plugin name="diff_drive_controller" filename="libgazebo_ros_diff_drive.so">
+      <ros>
+        <remapping>cmd_vel:=cmd_vel</remapping>
+        <remapping>odom:=odom</remapping>
+      </ros>
+      <update_rate>50</update_rate>
+      <left_joint>left_rear_wheel_joint</left_joint>
+      <right_joint>right_rear_wheel_joint</right_joint>
+      <wheel_separation>${wheel_separation}</wheel_separation>
+      <wheel_diameter>${2.0 * wheel_radius}</wheel_diameter>
+      <max_wheel_torque>30.0</max_wheel_torque>
+      <max_wheel_acceleration>3.0</max_wheel_acceleration>
+      <command_timeout>0.25</command_timeout>
+      <publish_odom>true</publish_odom>
+      <publish_odom_tf>true</publish_odom_tf>
+      <publish_wheel_tf>false</publish_wheel_tf>
+      <odometry_frame>odom</odometry_frame>
+      <robot_base_frame>base_footprint</robot_base_frame>
+      <!-- Leave odometry_source unset for broad Gazebo Classic compatibility. -->
+    </plugin>
+    <!-- Publish simulated wheel joint states so robot_state_publisher can produce wheel TF in RViz. -->
+    <plugin name="joint_state_publisher" filename="libgazebo_ros_joint_state_publisher.so">
+      <ros>
+        <remapping>~/out:=joint_states</remapping>
+      </ros>
+      <update_rate>50</update_rate>
+      <joint_name>left_rear_wheel_joint</joint_name>
+      <joint_name>right_rear_wheel_joint</joint_name>
+    </plugin>
+  </gazebo>
   <!-- Gazebo plugin for lidar simulation -->
   <xacro:sim_lidar/>

Commit message: progress forwards, physics better than before, Nav stack mostly working, has a weird issue lining up with goal orientation once it reaches the goal pose
Made-with: Cursor

File: src/create_robot/create_description/urdf/rectangular_robot.urdf.xacro (robot description, xacro)
@@ -33,6 +33,7 @@
   <xacro:property name="wheel_separation" value="0.57" />  <!-- Distance between rear wheels -->
   <!-- Note: Rear wheels are forward by one wheel radius (origin is between rear wheels) -->
-  <!-- Caster wheel properties -->
-  <xacro:property name="caster_radius" value="0.12" />
+  <!-- Caster: keep radius == wheel_radius so sphere center height matches rear axle height (level base).
+       If caster_radius < wheel_radius, the front sits low and the chassis pitches nose-down (and lidar tilts). -->
+  <xacro:property name="caster_radius" value="${wheel_radius}" />
   <xacro:property name="caster_mass" value="0.5" />
   <!-- Caster at front of robot (base extends from x=0 to x=base_length, center at base_length/2) -->
@@ -72,6 +73,4 @@
       <origin xyz="${x} ${y} ${z}" rpy="0 0 0"/>
       <axis xyz="${axis_xyz}"/>
-      <!-- Stronger damping to suppress residual idle creep in Gazebo Classic. -->
-      <dynamics damping="0.5" friction="0.0"/>
     </joint>
   </xacro:macro>
@@ -99,11 +98,4 @@
     </inertial>
   </link>
-  <!-- Add small body damping so the chassis settles at idle in simulation. -->
-  <gazebo reference="base_link">
-    <velocity_decay>
-      <linear>1.0</linear>
-      <angular>1.0</angular>
-    </velocity_decay>
-  </gazebo>
   <!-- Rear wheels for Gazebo diff-drive: keep both joint axes aligned (+Y) so forward cmd drives straight. -->
   <xacro:wheel name="left_rear_wheel" x="${wheel_radius}" y="${wheel_separation/2}" z="${wheel_radius}" axis_xyz="0 1 0"/>
@@ -133,36 +125,11 @@
     <parent link="base_link"/>
     <child link="front_caster_wheel"/>
-    <!-- Caster at front of robot, at ground level -->
-    <origin xyz="${caster_x_offset} 0 ${caster_radius}" rpy="0 0 0"/>
+    <!-- Sphere center at same z as rear wheel centers (wheel_radius) so all contacts lie on z=0 when base is level. -->
+    <origin xyz="${caster_x_offset} 0 ${wheel_radius}" rpy="0 0 0"/>
   </joint>
-  <!-- Front caster with moderate contact (avoid injecting forward creep). -->
+  <!-- Front caster: zero Coulomb friction (ideal ball; avoids scrub braking turns). -->
   <gazebo reference="front_caster_wheel">
-    <mu1>0.05</mu1>
-    <mu2>0.05</mu2>
-    <kp>1000000.0</kp>
-    <kd>1.0</kd>
-    <minDepth>0.001</minDepth>
-    <maxVel>0.0</maxVel>
-  </gazebo>
-  <!-- Rear drive wheel contact tuning: high traction, low slip. -->
-  <gazebo reference="left_rear_wheel">
-    <mu1>1.5</mu1>
-    <mu2>1.5</mu2>
-    <slip1>0.0</slip1>
-    <slip2>0.0</slip2>
-    <kp>1000000.0</kp>
-    <kd>1.0</kd>
-    <minDepth>0.001</minDepth>
-    <maxVel>0.0</maxVel>
-  </gazebo>
-  <gazebo reference="right_rear_wheel">
-    <mu1>1.5</mu1>
-    <mu2>1.5</mu2>
-    <slip1>0.0</slip1>
-    <slip2>0.0</slip2>
-    <kp>1000000.0</kp>
-    <kd>1.0</kd>
-    <minDepth>0.001</minDepth>
-    <maxVel>0.0</maxVel>
+    <mu1>0.0</mu1>
+    <mu2>0.0</mu2>
   </gazebo>
   <!-- Sweeping Wheel (parallel to floor - horizontal cylinder) -->
@@ -202,5 +169,5 @@
     <origin xyz="${wheel_radius} 0 0" rpy="0 0 0"/>
   </joint>
-  <!-- Keep lidar directly over rear axle (real robot mounting), raise height to reduce wheel returns. -->
+  <!-- Keep lidar directly over rear axle (real robot mounting). -->
   <xacro:lidar parent_link="base_link" x="${wheel_radius}" y="0" z="${base_height + 0.25}"/>
   <!-- Gazebo diff-drive for Classic simulation -->
@@ -218,5 +185,4 @@
       <max_wheel_torque>30.0</max_wheel_torque>
       <max_wheel_acceleration>3.0</max_wheel_acceleration>
-      <command_timeout>0.25</command_timeout>
       <publish_odom>true</publish_odom>
       <publish_odom_tf>true</publish_odom_tf>
