Commit message: Save robot logic and coverage assets

File: src/create_robot/create_description/urdf/rectangular_robot.urdf.xacro (robot description, xacro)
@@ -190,5 +190,13 @@
   </joint>
   <!-- Keep lidar directly over rear axle (real robot mounting). -->
-  <xacro:lidar parent_link="base_link" x="${wheel_radius}" y="0" z="${base_height + 0.25}"/>
+  <xacro:lidar parent_link="base_link" x="${wheel_radius + 0.11}" y="0" z="${base_height + 0.25}"/>
+  <!-- IMU frame for a chassis-mounted MPU-6050, centered and 0.15 m forward of the rear axle.
+       Assumes board axes match robot x-forward, y-left, z-up. -->
+  <link name="imu_link"/>
+  <joint name="imu_joint" type="fixed">
+    <parent link="base_link"/>
+    <child link="imu_link"/>
+    <origin xyz="${wheel_radius + 0.15} 0 ${base_height + 0.05}" rpy="0 0 0"/>
+  </joint>
   <!-- Gazebo diff-drive for Classic simulation -->
   <gazebo>
