Commit message: Still working sim with nav stack mostly figured out. Cranked up the lidars distance and that removed the issue where the robot would drift on the map. Not sure if that is a permenate solution
Made-with: Cursor

File: src/create_robot/create_description/urdf/lidar_gazebo.urdf.xacro (robot description, xacro)
@@ -19,5 +19,5 @@
           <range>
             <min>0.3</min>
-            <max>12</max>
+            <max>20</max>
           </range>
         </ray>

File: src/create_robot/create_description/urdf/rectangular_robot.urdf.xacro (robot description, xacro)
@@ -42,5 +42,6 @@
   <xacro:property name="sweep_wheel_radius" value="0.15" />
   <xacro:property name="sweep_wheel_length" value="0.03" />
-  <xacro:property name="sweep_wheel_mass" value="1.5" />
+  <!-- Non-physical visual marker only; Nav2 footprint handles avoidance envelope. -->
+  <xacro:property name="sweep_wheel_mass" value="0.0001" />
   <!-- Sweep wheel at front of robot -->
   <xacro:property name="sweep_wheel_x" value="${base_length}" />  <!-- Front edge of base -->
@@ -142,14 +143,9 @@
       <material name="orange"/>
     </visual>
-    <collision>
-      <origin xyz="0 0 0" rpy="0 0 0"/>
-      <geometry>
-        <cylinder radius="${sweep_wheel_radius}" length="${sweep_wheel_length}"/>
-      </geometry>
-    </collision>
+    <!-- No collision on purpose: keep this link out of Gazebo contact dynamics. -->
     <inertial>
       <origin xyz="0 0 0" rpy="0 0 0"/>
       <mass value="${sweep_wheel_mass}"/>
-      <inertia ixx="0.15" ixy="0" ixz="0" iyy="0.15" iyz="0" izz="0.15"/>
+      <inertia ixx="1e-6" ixy="0" ixz="0" iyy="1e-6" iyz="0" izz="1e-6"/>
     </inertial>
   </link>
@@ -185,4 +181,5 @@
       <max_wheel_torque>30.0</max_wheel_torque>
       <max_wheel_acceleration>3.0</max_wheel_acceleration>
+      <command_timeout>0.25</command_timeout>
       <publish_odom>true</publish_odom>
       <publish_odom_tf>true</publish_odom_tf>
