Commit message: Improve coordinated navigation robustness

File: src/create2_demo/urdf/rectangular_robot.urdf.xacro (robot description, xacro)
@@ -19,5 +19,5 @@
       <material name="blue"/>
     </visual>
-    <collision>
+    <collision name="base_link_collision">
       <origin xyz="${base_length / 2} 0 ${wheel_radius + base_height / 2}"/>
       <geometry><box size="${base_length} ${base_width} ${base_height}"/></geometry>
@@ -33,4 +33,18 @@
     <origin xyz="${wheel_radius} 0 0"/>
   </joint>
+  <!-- Report chassis impacts without treating normal wheel/ground contact as
+       a collision event.  The monitor records what the robot was doing and
+       what its LiDAR saw immediately before this sensor fired. -->
+  <gazebo reference="base_link">
+    <sensor name="chassis_contact_sensor" type="contact">
+      <always_on>true</always_on>
+      <update_rate>50</update_rate>
+      <contact><collision>base_link_collision</collision></contact>
+      <plugin name="chassis_contact_plugin" filename="libgazebo_ros_bumper.so">
+        <ros><remapping>bumper_states:=chassis_contacts</remapping></ros>
+        <frame_name>base_link</frame_name>
+      </plugin>
+    </sensor>
+  </gazebo>
   <xacro:macro name="drive_wheel" params="side y">
     <link name="${side}_rear_wheel">
@@ -40,5 +54,5 @@
         <material name="black"/>
       </visual>
-      <collision>
+      <collision name="${side}_rear_wheel_collision">
         <origin rpy="${pi / 2} 0 0"/>
         <geometry><cylinder radius="${wheel_radius}" length="${wheel_width}"/></geometry>
@@ -58,4 +72,13 @@
       <kp>1000000.0</kp><kd>100.0</kd>
       <maxVel>0.01</maxVel><minDepth>0.001</minDepth>
+      <sensor name="${side}_rear_wheel_contact_sensor" type="contact">
+        <always_on>true</always_on>
+        <update_rate>50</update_rate>
+        <contact><collision>${side}_rear_wheel_collision</collision></contact>
+        <plugin name="${side}_rear_wheel_contact_plugin" filename="libgazebo_ros_bumper.so">
+          <ros><remapping>bumper_states:=${side}_rear_wheel_contacts</remapping></ros>
+          <frame_name>${side}_rear_wheel</frame_name>
+        </plugin>
+      </sensor>
     </gazebo>
   </xacro:macro>
@@ -64,5 +87,5 @@
   <link name="front_caster_wheel">
     <visual><geometry><sphere radius="${wheel_radius}"/></geometry><material name="gray"/></visual>
-    <collision><geometry><sphere radius="${wheel_radius}"/></geometry></collision>
+    <collision name="front_caster_collision"><geometry><sphere radius="${wheel_radius}"/></geometry></collision>
     <inertial><mass value="0.5"/><inertia ixx="0.003" ixy="0" ixz="0" iyy="0.003" iyz="0" izz="0.003"/></inertial>
   </link>
@@ -76,4 +99,15 @@
     <kp>1000000.0</kp><kd>100.0</kd>
     <maxVel>0.01</maxVel><minDepth>0.001</minDepth>
+    <!-- The caster protrudes ahead of the chassis and can be the first robot
+         part to hit a wall. The logger filters its normal floor contact. -->
+    <sensor name="front_caster_contact_sensor" type="contact">
+      <always_on>true</always_on>
+      <update_rate>50</update_rate>
+      <contact><collision>front_caster_collision</collision></contact>
+      <plugin name="front_caster_contact_plugin" filename="libgazebo_ros_bumper.so">
+        <ros><remapping>bumper_states:=front_caster_contacts</remapping></ros>
+        <frame_name>front_caster_wheel</frame_name>
+      </plugin>
+    </sensor>
   </gazebo>
   <link name="sweeping_wheel">
@@ -99,5 +133,8 @@
   <gazebo reference="laser_frame">
     <sensor name="laser" type="ray">
-      <pose>0 0 0 0 0 0</pose><visualize>true</visualize><update_rate>10</update_rate>
+      <!-- Keep sensor activation independent of Gazebo rendering/client state. -->
+      <!-- Five hertz is above the two-hertz SLAM processing limit and divides
+           exactly into the 50 Hz odometry cadence without queuing unused scans. -->
+      <pose>0 0 0 0 0 0</pose><always_on>true</always_on><visualize>true</visualize><update_rate>5</update_rate>
       <ray>
         <scan><horizontal><samples>360</samples><resolution>1</resolution><min_angle>-${pi}</min_angle><max_angle>${pi}</max_angle></horizontal></scan>

File: src/create_robot/create_description/urdf/rectangular_robot.urdf.xacro (robot description, xacro)
@@ -133,4 +133,28 @@
     <mu1>0.0</mu1>
     <mu2>0.0</mu2>
+    <!-- Dampen the rigid sphere/ground contact.  Gazebo's stiff defaults can
+         inject vertical energy into a heavy three-contact-point chassis. -->
+    <kp>100000.0</kp>
+    <kd>100.0</kd>
+    <maxVel>0.05</maxVel>
+    <minDepth>0.001</minDepth>
+  </gazebo>
+  <!-- Driven wheels need predictable longitudinal contact and damped normal
+       contact; otherwise the diff-drive controller can excite chassis hop. -->
+  <gazebo reference="left_rear_wheel">
+    <mu1>1.0</mu1>
+    <mu2>1.0</mu2>
+    <kp>100000.0</kp>
+    <kd>100.0</kd>
+    <maxVel>0.05</maxVel>
+    <minDepth>0.001</minDepth>
+  </gazebo>
+  <gazebo reference="right_rear_wheel">
+    <mu1>1.0</mu1>
+    <mu2>1.0</mu2>
+    <kp>100000.0</kp>
+    <kd>100.0</kd>
+    <maxVel>0.05</maxVel>
+    <minDepth>0.001</minDepth>
   </gazebo>
   <!-- Sweeping Wheel (parallel to floor - horizontal cylinder) -->
